Commit message: grabbing code and changed in camera tracking ball

File: mybot_description/urdf/robot_model/bot.gazebo.xacro (robot description, xacro)
@@ -63,5 +63,5 @@
       <wheelDiameter>0.4</wheelDiameter>
       <wheelAcceleration>1</wheelAcceleration>
-      <wheelTorque>1000</wheelTorque>
+      <wheelTorque>10</wheelTorque>
       <rosDebugLevel>na</rosDebugLevel>
     </plugin>

File: mybot_description/urdf/robot_model/bot.urdf.xacro (robot description, xacro)
@@ -4,6 +4,6 @@
   <xacro:include filename="$(find mybot_description)/urdf/robot_model/bot.gazebo.xacro"/>
   <xacro:property name="base_mass" value= "6" />
-  <xacro:property name="wheel_mass" value= "0.05" />
-  <xacro:property name="default_mass" value= "0.01" />
+  <xacro:property name="wheel_mass" value= "0.01" />
+  <xacro:property name="default_mass" value= "0.0001" />
    <xacro:property name="base_x" value= "0.6" />
    <xacro:property name="base_y" value="0.6" />
@@ -103,5 +103,5 @@
     <child link="slider"/>
     <axis xyz="0 0 1"/>
-    <limit effort="100000.0" lower="${-slider_z}" upper="0" velocity="0.5"/>
+    <limit effort="1000.0" lower="${-slider_z}" upper="0" velocity="0.5"/>
     <origin xyz="${arm_base_x*0.5 + slider_z} ${arm_base_y*0.5 + arm_y*0.5} 0" rpy="0 1.57 0"/>
   </joint>
@@ -131,5 +131,5 @@
     <type>transmission_interface/SimpleTransmission</type>
     <actuator name="slider_motor">
-      <mechanicalReduction>50</mechanicalReduction>
+      <mechanicalReduction>1</mechanicalReduction>
     <hardwareInterface>EffortJointInterface</hardwareInterface>
     </actuator>
@@ -143,5 +143,5 @@
     <child link="arm"/>
     <axis xyz="0 1 0"/>
-    <limit effort="1000.0" lower="0.0" upper="1.57" velocity="0.5"/>
+    <limit effort="1000.0" lower="0.0" upper="1.57" velocity="0.1"/>
     <origin xyz="0 0 0" rpy="0 -1.57 0"/>
   </joint>
