Commit message: navigation to goal with ros navigations stack added

File: mybot_description/urdf/turtlebot/turtlebot3_waffle.urdf.xacro (robot description, xacro)
@@ -4,8 +4,8 @@
   <xacro:include filename="$(find mybot_description)/urdf/turtlebot/turtlebot3_waffle.gazebo.xacro"/>
    <xacro:property name="arm_mount_height" value="0.1" />
-   <xacro:property name="arm_len" value="0.6" />
+   <xacro:property name="arm_len" value="0.3" />
    <xacro:property name="arm_width" value="0.02" />
    <xacro:property name="arm_thick" value="0.01" />
-   <xacro:property name="arm_dist" value="0.5" />
+   <xacro:property name="arm_dist" value="0.3" />
    <xacro:property name="camera_size" value="${arm_width*0.8}"/>
    <xacro:property name="default_mas" value="0.005" />

Commit message: testing

File: mybot_description/urdf/turtlebot/turtlebot3_waffle.urdf.xacro (robot description, xacro)
@@ -3,7 +3,7 @@
   <xacro:include filename="$(find mybot_description)/urdf/turtlebot/common_properties.xacro"/>
   <xacro:include filename="$(find mybot_description)/urdf/turtlebot/turtlebot3_waffle.gazebo.xacro"/>
-   <xacro:property name="arm_mount_height" value="0.1" />
+   <xacro:property name="arm_mount_height" value="0.05" />
    <xacro:property name="arm_len" value="0.3" />
-   <xacro:property name="arm_width" value="0.02" />
+   <xacro:property name="arm_width" value="0.08" />
    <xacro:property name="arm_thick" value="0.01" />
    <xacro:property name="arm_dist" value="0.3" />
